File: PCB - Copy/LED&Buzzer.kicad_sch (KiCad schematic)
At the start: 13 parts, among them Q5 BC547

Commit message: ADDED VALUES
Parts:
- BZ1: footprint Buzzer_Beeper:Buzzer_12x9.5RM7.6 -> myLib:Buzzer_12x9.5RM7.6
- D3, D4, D5, D6, D7, D8: footprint LED_THT:LED_D3.0mm -> MyLib:LED_D3.0mm
Changed lines of the file:
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@@
     (property "Reference" "D3" (id 0) (at 95.4278 78.613 0))
     (property "Value" "LED" (id 1) (at 95.4278 80.9244 0))
-    (property "Footprint" "LED_THT:LED_D3.0mm" (id 2) (at 95.25 85.09 0)
+    (property "Footprint" "MyLib:LED_D3.0mm" (id 2) (at 95.25 85.09 0)
       (effects (font (size 1.27 1.27)) hide)
     )
@@
       (effects (font (size 1.27 1.27)) (justify left))
     )
-    (property "Footprint" "Buzzer_Beeper:Buzzer_12x9.5RM7.6" (id 2) (at 151.765 73.66 90)
+    (property "Footprint" "myLib:Buzzer_12x9.5RM7.6" (id 2) (at 151.765 73.66 90)
       (effects (font (size 1.27 1.27)) hide)
     )
@@
     (property "Reference" "D4" (id 0) (at 95.4278 97.663 0))
     (property "Value" "LED" (id 1) (at 95.4278 99.9744 0))
-    (property "Footprint" "LED_THT:LED_D3.0mm" (id 2) (at 95.25 104.14 0)
+    (property "Footprint" "MyLib:LED_D3.0mm" (id 2) (at 95.25 104.14 0)
       (effects (font (size 1.27 1.27)) hide)
     )
@@
     (property "Reference" "D5" (id 0) (at 95.4278 115.443 0))
     (property "Value" "LED" (id 1) (at 95.4278 117.7544 0))
-    (property "Footprint" "LED_THT:LED_D3.0mm" (id 2) (at 95.25 121.92 0)
+    (property "Footprint" "MyLib:LED_D3.0mm" (id 2) (at 95.25 121.92 0)
       (effects (font (size 1.27 1.27)) hide)
     )
@@
     (property "Reference" "D6" (id 0) (at 198.2978 79.883 0))
     (property "Value" "LED" (id 1) (at 198.2978 82.1944 0))
-    (property "Footprint" "LED_THT:LED_D3.0mm" (id 2) (at 198.12 86.36 0)
+    (property "Footprint" "MyLib:LED_D3.0mm" (id 2) (at 198.12 86.36 0)
       (effects (font (size 1.27 1.27)) hide)
     )
@@
     (property "Reference" "D7" (id 0) (at 198.2978 91.313 0))
     (property "Value" "LED" (id 1) (at 198.2978 93.6244 0))
-    (property "Footprint" "LED_THT:LED_D3.0mm" (id 2) (at 198.12 97.79 0)
+    (property "Footprint" "MyLib:LED_D3.0mm" (id 2) (at 198.12 97.79 0)
       (effects (font (size 1.27 1.27)) hide)
     )
@@
     (property "Reference" "D8" (id 0) (at 198.2978 101.473 0))
     (property "Value" "LED" (id 1) (at 198.2978 103.7844 0))
-    (property "Footprint" "LED_THT:LED_D3.0mm" (id 2) (at 198.12 107.95 0)
-      (effects (font (size 1.27 1.27)) hide)
-    )
+    (property "Footprint" "MyLib:LED_D3.0mm" (id 2) (at 198.12 107.95 0)
+      (effects (font (size 1.27 1.27)) hide)
+    )
