File: PCB - Copy/Power.kicad_sch (KiCad schematic)
At the start: 13 parts, among them J3 Conn_01x02, U2 L7805

Commit message: ADDED VALUES
Parts:
- C4: footprint Capacitor_THT:CP_Radial_D10.0mm_P5.00mm -> myLib:CP_Radial_D10.0mm_P5.00mm
- C6, C7: footprint Capacitor_THT:CP_Radial_D5.0mm_P2.50mm -> myLib:CP_Radial_D5.0mm_P2.50mm
- R16: value 330R -> 56K
- R17: value 330R -> 15K
- U2: footprint Package_TO_SOT_THT:TO-220-3_Vertical -> myLib:TO-220-3_Vertical
Changed lines of the file:
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@@
       (effects (font (size 1.27 1.27)) (justify left))
     )
-    (property "Footprint" "Capacitor_THT:CP_Radial_D10.0mm_P5.00mm" (id 2) (at 101.6 95.25 0)
+    (property "Footprint" "myLib:CP_Radial_D10.0mm_P5.00mm" (id 2) (at 101.6 95.25 0)
       (effects (font (size 1.27 1.27)) hide)
     )
@@
     (property "Reference" "U2" (id 0) (at 120.65 77.6732 0))
     (property "Value" "L7805" (id 1) (at 120.65 79.9846 0))
-    (property "Footprint" "Package_TO_SOT_THT:TO-220-3_Vertical" (id 2) (at 121.285 87.63 0)
+    (property "Footprint" "myLib:TO-220-3_Vertical" (id 2) (at 121.285 87.63 0)
       (effects (font (size 1.27 1.27) italic) (justify left) hide)
     )
@@
       (effects (font (size 1.27 1.27)) (justify left))
     )
-    (property "Footprint" "Capacitor_THT:CP_Radial_D5.0mm_P2.50mm" (id 2) (at 148.59 95.25 0)
+    (property "Footprint" "myLib:CP_Radial_D5.0mm_P2.50mm" (id 2) (at 148.59 95.25 0)
       (effects (font (size 1.27 1.27)) hide)
     )
@@
       (effects (font (size 1.27 1.27)) (justify left))
     )
-    (property "Value" "330R" (id 1) (at 67.818 43.053 0)
+    (property "Value" "56K" (id 1) (at 67.818 43.053 0)
       (effects (font (size 1.27 1.27)) (justify left))
     )
@@
       (effects (font (size 1.27 1.27)) (justify left))
     )
-    (property "Value" "330R" (id 1) (at 67.818 54.483 0)
+    (property "Value" "15K" (id 1) (at 67.818 54.483 0)
       (effects (font (size 1.27 1.27)) (justify left))
     )
@@
       (effects (font (size 1.27 1.27)) (justify left))
     )
-    (property "Footprint" "Capacitor_THT:CP_Radial_D5.0mm_P2.50mm" (id 2) (at 88.9 53.34 0)
+    (property "Footprint" "myLib:CP_Radial_D5.0mm_P2.50mm" (id 2) (at 88.9 53.34 0)
       (effects (font (size 1.27 1.27)) hide)
     )
