File: PCB - Copy/Sensors.kicad_sch (KiCad schematic)
At the start: 17 parts, among them J1 Conn_01x04, J4 Conn_01x02, Q1 BC547

Commit message: ADDED VALUES
Parts:
- J1: footprint TerminalBlock:TerminalBlock_bornier-4_P5.08mm -> myLib:TerminalBlock_bornier-4_P5.08mm
- R19: value 330R -> 10K
- R2: value 330R -> 10K; footprint Resistor_THT:R_Axial_DIN0207_L6.3mm_D2.5mm_P10.16mm_Horizontal -> MyLib:R_Axial_DIN0207_L6.3mm_D2.5mm_P10.16mm_Horizontal
- R3, R4: value 330R -> 1K
- R5: value 10k -> 10K; footprint Resistor_THT:R_Axial_DIN0207_L6.3mm_D2.5mm_P10.16mm_Horizontal -> MyLib:R_Axial_DIN0207_L6.3mm_D2.5mm_P10.16mm_Horizontal
- R7: value 100k -> 68K
Changed lines of the file:
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@@
       (effects (font (size 1.27 1.27)) (justify left))
     )
-    (property "Value" "330R" (id 1) (at 59.817 85.598 0)
+    (property "Value" "1K" (id 1) (at 59.817 85.598 0)
       (effects (font (size 1.27 1.27)) (justify left))
     )
@@
     (property "Reference" "J1" (id 0) (at 35.1028 92.075 0))
     (property "Value" "Conn_01x04" (id 1) (at 35.1028 89.7636 0))
-    (property "Footprint" "TerminalBlock:TerminalBlock_bornier-4_P5.08mm" (id 2) (at 33.02 81.28 0)
+    (property "Footprint" "myLib:TerminalBlock_bornier-4_P5.08mm" (id 2) (at 33.02 81.28 0)
       (effects (font (size 1.27 1.27)) hide)
     )
@@
       (effects (font (size 1.27 1.27)) (justify left))
     )
-    (property "Value" "330R" (id 1) (at 62.103 122.682 0)
-      (effects (font (size 1.27 1.27)) (justify left))
-    )
-    (property "Footprint" "Resistor_THT:R_Axial_DIN0207_L6.3mm_D2.5mm_P10.16mm_Horizontal" (id 2) (at 60.96 126.238 90)
+    (property "Value" "10K" (id 1) (at 62.103 122.682 0)
+      (effects (font (size 1.27 1.27)) (justify left))
+    )
+    (property "Footprint" "MyLib:R_Axial_DIN0207_L6.3mm_D2.5mm_P10.16mm_Horizontal" (id 2) (at 60.96 126.238 90)
       (effects (font (size 1.27 1.27)) hide)
     )
@@
       (effects (font (size 1.27 1.27)) (justify left))
     )
-    (property "Value" "330R" (id 1) (at 68.453 93.218 0)
+    (property "Value" "10K" (id 1) (at 68.453 93.218 0)
       (effects (font (size 1.27 1.27)) (justify left))
     )
@@
       (effects (font (size 1.27 1.27)) (justify left))
     )
-    (property "Value" "10k" (id 1) (at 66.167 54.737 0)
-      (effects (font (size 1.27 1.27)) (justify left))
-    )
-    (property "Footprint" "Resistor_THT:R_Axial_DIN0207_L6.3mm_D2.5mm_P10.16mm_Horizontal" (id 2) (at 69.723 55.88 90)
+    (property "Value" "10K" (id 1) (at 66.167 54.737 0)
+      (effects (font (size 1.27 1.27)) (justify left))
+    )
+    (property "Footprint" "MyLib:R_Axial_DIN0207_L6.3mm_D2.5mm_P10.16mm_Horizontal" (id 2) (at 69.723 55.88 90)
       (effects (font (size 1.27 1.27)) hide)
     )
@@
       (effects (font (size 1.27 1.27)) (justify left))
     )
-    (property "Value" "100k" (id 1) (at 68.453 133.858 0)
+    (property "Value" "68K" (id 1) (at 68.453 133.858 0)
       (effects (font (size 1.27 1.27)) (justify left))
     )
@@
       (effects (font (size 1.27 1.27)) (justify left))
     )
-    (property "Value" "330R" (id 1) (at 61.087 48.768 0)
-      (effects (font (size 1.27 1.27)) (justify left))
-    )
+    (property "Value" "1K" (id 1) (at 61.087 48.768 0)
+      (effects (font (size 1.27 1.27)) (justify left))
+    )
