File: PCB - Copy2/Sensors.kicad_sch (KiCad schematic)
At the start: 17 parts, among them J1 Conn_01x04, J4 Conn_01x02, Q1 BC547

Commit message: nedd to connect ground
Parts:
- Q1: footprint Package_TO_SOT_THT:TO-92_Inline -> Package_TO_SOT_THT:TO-92L_Wide
Changed lines of the file:
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@@
       (effects (font (size 1.27 1.27)) (justify left))
     )
-    (property "Footprint" "Package_TO_SOT_THT:TO-92_Inline" (id 2) (at 90.17 126.365 0)
+    (property "Footprint" "Package_TO_SOT_THT:TO-92L_Wide" (id 2) (at 90.17 126.365 0)
       (effects (font (size 1.27 1.27) italic) (justify left) hide)
     )
